Commit message: mobile robot model is done

File: src/mastering_ros_robot_description_pkg/urdf/diff_wheeled_robot.xacro (robot description, xacro)
@@ -1,10 +1,6 @@
-<?xml version="1.0" ?>
-<!-- =================================================================================== -->
-<!-- |    This document was autogenerated by xacro from diff_wheeled_robot.xacro       | -->
-<!-- |    EDITING THIS FILE BY HAND IS NOT RECOMMENDED                                 | -->
-<!-- =================================================================================== -->
-<robot name="differential_wheeled_robot">
-  <!-- in kg-->
-  <!-- Defining the colors used in this robot -->
+<?xml version="1.0"?>
+<robot name="differential_wheeled_robot" xmlns:xacro="http://ros.org/wiki/xacro">
+  <xacro:include filename="$(find mastering_ros_robot_description_pkg)/urdf/wheel.urdf.xacro" />
+<!-- Defining the colors used in this robot -->
   <material name="Black">
     <color rgba="0.0 0.0 0.0 1.0"/>
@@ -19,20 +15,52 @@
     <color rgba="0.0 0.0 0.8 1.0"/>
   </material>
-  <!-- in kg-->
-  <!-- in kg-->
-   --&gt;
+  <!-- PROPERTY LIST -->
+  <!--All units in m-kg-s-radians unit system -->
+  <xacro:property name="M_PI" value="3.1415926535897931" />
+  <xacro:property name="M_PI_2" value="1.570796327" />
+  <xacro:property name="DEG_TO_RAD" value="0.017453293" />
+  <!-- Main body radius and height -->
+  <!-- Main Body Cylinder base   -->
+  <xacro:property name="base_height" value="0.02" />
+  <xacro:property name="base_radius" value="0.15" />
+  <xacro:property name="base_mass" value="5.0" /> <!-- in kg-->
+  <!-- caster wheel radius and height -->
+  <!-- caster wheel mass -->
+  <xacro:property name="caster_f_height" value="0.04" />
+  <xacro:property name="caster_f_radius" value="0.025" />
+  <xacro:property name="caster_f_mass" value="0.5" />
+  <!-- caster wheel radius and height -->
+  <!-- caster wheel mass -->
+  <xacro:property name="caster_b_height" value="0.04" />
+  <xacro:property name="caster_b_radius" value="0.025" />
+  <xacro:property name="caster_b_mass" value="0.5" /> <!-- in kg-->
+  <!-- Wheels -->
+  <xacro:property name="wheel_mass" value="2.5" /> --> <!-- in kg-->
+  <xacro:property name="base_x_origin_to_wheel_origin" value="0.25" />
+  <xacro:property name="base_y_origin_to_wheel_origin" value="0.3" />
+  <xacro:property name="base_z_origin_to_wheel_origin" value="0.0" />
+  <!-- Hokuyo Laser scanner -->
+  <xacro:property name="hokuyo_size" value="0.05" />
+  <!-- Macro for calculating inertia of cylinder -->
+  <xacro:macro name="cylinder_inertia" params="m r h">
+    <inertia  ixx="${m*(3*r*r+h*h)/12}" ixy = "0" ixz = "0"
+              iyy="${m*(3*r*r+h*h)/12}" iyz = "0"
+              izz="${m*r*r/2}" />
+  </xacro:macro>
   <!-- BASE-FOOTPRINT -->
   <!-- base_footprint is a fictitious link(frame) that is on the ground right below base_link origin -->
   <link name="base_footprint">
     <inertial>
-      <mass value="0.0001"/>
-      <origin xyz="0 0 0"/>
-      <inertia ixx="0.0001" ixy="0.0" ixz="0.0" iyy="0.0001" iyz="0.0" izz="0.0001"/>
+      <mass value="0.0001" />
+      <origin xyz="0 0 0" />
+      <inertia ixx="0.0001" ixy="0.0" ixz="0.0"
+          iyy="0.0001" iyz="0.0"
+          izz="0.0001" />
     </inertial>
     <visual>
-      <origin rpy="0 0 0" xyz="0 0 0"/>
-      <geometry>
-        <box size="0.001 0.001 0.001"/>
-      </geometry>
+        <origin xyz="0 0 0" rpy="0 0 0" />
+        <geometry>
+            <box size="0.001 0.001 0.001" />
+        </geometry>
     </visual>
   </link>
@@ -41,26 +69,28 @@
   </gazebo>
   <joint name="base_footprint_joint" type="fixed">
-    <origin rpy="0 0 0" xyz="0 0 0.04"/>
+    <origin xyz="0 0 ${wheel_radius - base_z_origin_to_wheel_origin}" rpy="0 0 0" />
     <parent link="base_footprint"/>
-    <child link="base_link"/>
+    <child link="base_link" />
   </joint>
   <link name="base_link">
     <inertial>
-      <mass value="5.0"/>
-      <origin xyz="0 0 0"/>
-      <inertia ixx="0.0001" ixy="0.0" ixz="0.0" iyy="0.0001" iyz="0.0" izz="0.0001"/>
-      <cylinder_inertia h="0.02" m="5.0" r="0.15"/>
+      <mass value="${base_mass}" />
+      <origin xyz="0 0 0" />
+      <inertia ixx="0.0001" ixy="0.0" ixz="0.0"
+          iyy="0.0001" iyz="0.0"
+          izz="0.0001" />
+      <cylinder_inertia  m="${base_mass}" r="${base_radius}" h="${base_height}" />
     </inertial>
     <visual>
-      <origin rpy="0 0 0" xyz="0 0 0"/>
+      <origin xyz="0 0 0" rpy="0 0 0" />
       <geometry>
-        <cylinder length="0.02" radius="0.15"/>
+          <cylinder length="${base_height}" radius="${base_radius}" />
       </geometry>
-      <material name="White"/>
+      <material name="White" />
     </visual>
     <collision>
-      <origin rpy="0 0 0 " xyz="0 0 0"/>
+      <origin xyz="0 0 0" rpy="0 0 0 " />
       <geometry>
-        <cylinder length="0.02" radius="0.15"/>
+          <cylinder length="${base_height}" radius="${base_radius}" />
       </geometry>
     </collision>
@@ -72,26 +102,28 @@
   <link name="caster_front_link">
     <visual>
-      <origin rpy="1.5707963267948966 0 0" xyz="0 0.02 0"/>
+      <origin xyz="0 0.02 0" rpy="${M_PI/2} 0 0" />
       <geometry>
-        <sphere radius="0.025"/>
+				<sphere radius="${caster_f_radius}" />
       </geometry>
-      <material name="Black"/>
+      <material name="Black" />
     </visual>
     <collision>
       <geometry>
-        <sphere radius="0.025"/>
+				<sphere radius="${caster_f_radius}" />
       </geometry>
-      <origin rpy="1.5707963267948966 0 0" xyz="0 0.02 0"/>
+    <origin xyz="0 0.02 0" rpy="${M_PI/2} 0 0" />
     </collision>
     <inertial>
-      <mass value="0.5"/>
-      <origin xyz="0 0 0"/>
-      <inertia ixx="0.001" ixy="0.0" ixz="0.0" iyy="0.001" iyz="0.0" izz="0.001"/>
+      <mass value="${caster_f_mass}" />
+      <origin xyz="0 0 0" />
+      <inertia ixx="0.001" ixy="0.0" ixz="0.0"
+               iyy="0.001" iyz="0.0"
+               izz="0.001" />
     </inertial>
   </link>
-  <joint name="caster_front_joint" type="fixed">
+	<joint name="caster_front_joint" type="fixed">
     <parent link="base_link"/>
     <child link="caster_front_link"/>
-    <origin rpy="-1.5707963267948966 0 0" xyz="0.115 0.0 0.007"/>
+    <origin xyz="0.115 0.0 0.007" rpy="${-M_PI/2} 0 0"/>
   </joint>
   <gazebo reference="caster_front_link">
@@ -99,21 +131,23 @@
   </gazebo>
   <link name="caster_back_link">
-    <visual>
-      <origin rpy="1.5707963267948966 0 0" xyz="0.02 0.02 0 "/>
-      <geometry>
-        <sphere radius="0.025"/>
-      </geometry>
-      <material name="Black"/>
-    </visual>
-    <collision>
-      <geometry>
-        <sphere radius="0.025"/>
-      </geometry>
-      <origin rpy="1.5707963267948966 0 0" xyz="0 0.02 0 "/>
+  <visual>
+    <origin xyz="0.02 0.02 0 " rpy="${M_PI/2} 0 0" />
+    <geometry>
+			<sphere radius="${caster_b_radius}" />
+    </geometry>
+    <material name="Black" />
+  </visual>
+  <collision>
+    <geometry>
+			<sphere radius="${caster_b_radius}" />
+     </geometry>
+     <origin xyz="0 0.02 0 " rpy="${M_PI/2} 0 0" />
     </collision>
     <inertial>
-      <mass value="0.5"/>
-      <origin xyz="0 0 0"/>
-      <inertia ixx="0.001" ixy="0.0" ixz="0.0" iyy="0.001" iyz="0.0" izz="0.001"/>
+      <mass value="${caster_b_mass}" />
+      <origin xyz="0 0 0" />
+      <inertia ixx="0.001" ixy="0.0" ixz="0.0"
+               iyy="0.001" iyz="0.0"
+               izz="0.001" />
     </inertial>
   </link>
@@ -121,125 +155,33 @@
     <parent link="base_link"/>
     <child link="caster_back_link"/>
-    <origin rpy="-1.5707963267948966 0 0" xyz="-0.135 0.0 0.009"/>
+    <origin xyz="-0.135 0.0 0.009" rpy="${-M_PI/2} 0 0"/>
   </joint>
   <gazebo reference="caster_back_link">
-    <turnGravityOff>false</turnGravityOff>
+   <turnGravityOff>false</turnGravityOff>
   </gazebo>
-  <!--fb : front, back ; lr: left, right -->
-  <link name="front_right_wheel">
-    <visual>
-      <origin rpy="1.5707963267948966 0  0 " xyz="0 0 0"/>
-      <geometry>
-        <cylinder length="0.02" radius="0.04"/>
-      </geometry>
-      <material name="DarkGray"/>
-    </visual>
-    <collision>
-      <origin rpy="1.5707963267948966 0 0 " xyz="0 0 0"/>
-      <geometry>
-        <cylinder length="0.02" radius="0.04"/>
-      </geometry>
-    </collision>
-    <inertial>
-      <mass value="2.5"/>
-      <origin xyz="0 0 0"/>
-      <cylinder_inertia h="0.02" m="2.5" r="0.04"/>
-    </inertial>
-  </link>
-  <gazebo reference="front_right_wheel">
-    <mu1 value="1.0"/>
-    <mu2 value="1.0"/>
-    <kp value="10000000.0"/>
-    <kd value="1.0"/>
-    <fdir1 value="1 0 0"/>
-    <material>Gazebo/Grey</material>
-    <turnGravityOff>false</turnGravityOff>
-  </gazebo>
-  <joint name="front_right_wheel_joint" type="continuous">
-    <parent link="base_link"/>
-    <child link="front_right_wheel"/>
-    <origin rpy="0 0 0" xyz="0.0 0.15 0.0"/>
-    <axis rpy="0 0 0" xyz="0 1 0"/>
-    <limit effort="100" velocity="100"/>
-    <joint_properties damping="0.0" friction="0.0"/>
-  </joint>
-  <!-- Transmission is important to link the joints and the controller -->
-  <transmission name="front_right_wheel_joint_trans">
-    <type>transmission_interface/SimpleTransmission</type>
-    <joint name="front_right_wheel_joint"/>
-    <actuator name="front_right_wheel_joint_motor">
-      <hardwareInterface>EffortJointInterface</hardwareInterface>
-      <mechanicalReduction>1</mechanicalReduction>
-    </actuator>
-  </transmission>
-  <!--fb : front, back ; lr: left, right -->
-  <link name="front_left_wheel">
-    <visual>
-      <origin rpy="1.5707963267948966 0  0 " xyz="0 0 0"/>
-      <geometry>
-        <cylinder length="0.02" radius="0.04"/>
-      </geometry>
-      <material name="DarkGray"/>
-    </visual>
-    <collision>
-      <origin rpy="1.5707963267948966 0 0 " xyz="0 0 0"/>
-      <geometry>
-        <cylinder length="0.02" radius="0.04"/>
-      </geometry>
-    </collision>
-    <inertial>
-      <mass value="2.5"/>
-      <origin xyz="0 0 0"/>
-      <cylinder_inertia h="0.02" m="2.5" r="0.04"/>
-    </inertial>
-  </link>
-  <gazebo reference="front_left_wheel">
-    <mu1 value="1.0"/>
-    <mu2 value="1.0"/>
-    <kp value="10000000.0"/>
-    <kd value="1.0"/>
-    <fdir1 value="1 0 0"/>
-    <material>Gazebo/Grey</material>
-    <turnGravityOff>false</turnGravityOff>
-  </gazebo>
-  <joint name="front_left_wheel_joint" type="continuous">
-    <parent link="base_link"/>
-    <child link="front_left_wheel"/>
-    <origin rpy="0 0 0" xyz="0.0 -0.15 0.0"/>
-    <axis rpy="0 0 0" xyz="0 1 0"/>
-    <limit effort="100" velocity="100"/>
-    <joint_properties damping="0.0" friction="0.0"/>
-  </joint>
-  <!-- Transmission is important to link the joints and the controller -->
-  <transmission name="front_left_wheel_joint_trans">
-    <type>transmission_interface/SimpleTransmission</type>
-    <joint name="front_left_wheel_joint"/>
-    <actuator name="front_left_wheel_joint_motor">
-      <hardwareInterface>EffortJointInterface</hardwareInterface>
-      <mechanicalReduction>1</mechanicalReduction>
-    </actuator>
-  </transmission>
-  <gazebo>
-    <plugin filename="libgazebo_ros_diff_drive.so" name="differential_drive_controller">
-      <legacyMode>true</legacyMode>
-      <rosDebugLevel>Debug</rosDebugLevel>
-      <publishWheelTF>false</publishWheelTF>
-      <robotNamespace>/</robotNamespace>
-      <publishTf>1</publishTf>
-      <publishWheelJointState>false</publishWheelJointState>
-      <alwaysOn>true</alwaysOn>
-      <updateRate>100.0</updateRate>
-      <leftJoint>front_left_wheel_joint</leftJoint>
-      <rightJoint>front_right_wheel_joint</rightJoint>
-      <wheelSeparation>0.3</wheelSeparation>
-      <wheelDiameter>0.08</wheelDiameter>
-      <broadcastTF>1</broadcastTF>
-      <wheelTorque>30</wheelTorque>
-      <wheelAcceleration>1.8</wheelAcceleration>
-      <commandTopic>cmd_vel</commandTopic>
-      <odometryFrame>odom</odometryFrame>
-      <odometryTopic>odom</odometryTopic>
-      <robotBaseFrame>base_footprint</robotBaseFrame>
-    </plugin>
+  <xacro:wheel fb="front" lr="right" parent="base_link" translateX="0" translateY="-0.5" flipY="1"/>
+	<xacro:wheel fb="front" lr="left" parent="base_link" translateX="0" translateY="0.5" flipY="1"/>
+	<gazebo>
+  	<plugin name="differential_drive_controller" filename="libgazebo_ros_diff_drive.so">
+	    <legacyMode>true</legacyMode>
+	    <rosDebugLevel>Debug</rosDebugLevel>
+	    <publishWheelTF>false</publishWheelTF>
+	    <robotNamespace>/</robotNamespace>
+	    <publishTf>1</publishTf>
+	    <publishWheelJointState>false</publishWheelJointState>
+	    <alwaysOn>true</alwaysOn>
+	    <updateRate>100.0</updateRate>
+	    <leftJoint>front_left_wheel_joint</leftJoint>
+	    <rightJoint>front_right_wheel_joint</rightJoint>
+	    <wheelSeparation>${2*base_radius}</wheelSeparation>
+	    <wheelDiameter>${2*wheel_radius}</wheelDiameter>
+	    <broadcastTF>1</broadcastTF>
+	    <wheelTorque>30</wheelTorque>
+	    <wheelAcceleration>1.8</wheelAcceleration>
+	    <commandTopic>cmd_vel</commandTopic>
+	    <odometryFrame>odom</odometryFrame>
+	    <odometryTopic>odom</odometryTopic>
+	    <robotBaseFrame>base_footprint</robotBaseFrame>
+   </plugin>
   </gazebo>
 </robot>
